File: CreditCard/CreditCard.kicad_pcb (KiCad board)
At the start: 2 copper layers, 85 x 50 mm, 0 parts

Commit message: début
début sch
Parts:
- added 3VTP1: TP, TestPoint:TestPoint_Pad_D1.5mm, F.Cu at (-55.2, 76.5)
- added C1: 0.1uF, Capacitor_SMD:C_0603_1608Metric, F.Cu at (-54.9, 58.9)
- added C10: 0.1uF, Capacitor_SMD:C_0603_1608Metric, F.Cu at (-60.9, 34.3)
- added C11: 0.1uF, Capacitor_SMD:C_0603_1608Metric, F.Cu at (-60.9, 36.8)
- added C12: 12pF, Capacitor_SMD:C_0603_1608Metric, F.Cu at (-54.9, 66.4)
- added C13: 4.7uF, Capacitor_SMD:C_0805_2012Metric, F.Cu at (-37.5, 50.0)
- added C14: 1uF, Capacitor_SMD:C_0603_1608Metric, F.Cu at (-54.9, 36.8)
- added C15: 4.7uF, Capacitor_SMD:C_0805_2012Metric, F.Cu at (-37.5, 53.0)
- added C16: 100n, Capacitor_SMD:C_0603_1608Metric, F.Cu at (-54.9, 39.3)
- added C17: 12pF, Capacitor_SMD:C_0603_1608Metric, F.Cu at (-54.9, 68.9)
- added C18: 0.1uF, Capacitor_SMD:C_0603_1608Metric, F.Cu at (-60.9, 39.3)
- added C19: 0.1uF, Capacitor_SMD:C_0603_1608Metric, F.Cu at (-60.9, 41.8)
- added C2: 1uF, Capacitor_SMD:C_0603_1608Metric, F.Cu at (-54.9, 61.4)
- added C20: 0.1uF, Capacitor_SMD:C_0603_1608Metric, F.Cu at (-60.9, 44.3)
- added C21: 0.1uF, Capacitor_SMD:C_0603_1608Metric, F.Cu at (-60.9, 46.8)
- added C3: 4.7uF, Capacitor_SMD:C_0805_2012Metric, F.Cu at (-37.5, 44.0)
- added C4: 4.7uF, Capacitor_SMD:C_0805_2012Metric, F.Cu at (-37.5, 47.0)
- added C7: 22uF, Capacitor_SMD:C_1206_3216Metric, F.Cu at (-50.1, 52.1)
- added C8: 0.1uF, Capacitor_SMD:C_0603_1608Metric, F.Cu at (-54.9, 34.3)
- added C9: 0.1uF, Capacitor_SMD:C_0603_1608Metric, F.Cu at (-54.9, 63.9)
- added D1: LED, LED_SMD:LED_0805_2012Metric, F.Cu at (-42.0, 44.0)
- added D2: LED, LED_SMD:LED_0805_2012Metric, F.Cu at (-42.0, 47.1)
- added D3: LED, LED_SMD:LED_0805_2012Metric, F.Cu at (-42.0, 50.1)
- added D5: D_TVS, Diode_SMD:D_SOD-323_HandSoldering, F.Cu at (-39.1, 39.0)
- added F1: ~, CommonLib_HORUS:GOLD_FINGERS, F.Cu at (-46.9, 58.7)
- added F2: ~, CommonLib_HORUS:GOLD_FINGERS, F.Cu at (-46.9, 61.0)
- added F4: ~, CommonLib_HORUS:GOLD_FINGERS, F.Cu at (-46.9, 63.2)
- added F5: ~, CommonLib_HORUS:GOLD_FINGERS, F.Cu at (-46.9, 65.5)
- added F6: ~, CommonLib_HORUS:GOLD_FINGERS, F.Cu at (-46.9, 67.7)
- added F7: ~, CommonLib_HORUS:GOLD_FINGERS, F.Cu at (-39.7, 34.2)
- added F8: ~, CommonLib_HORUS:GOLD_FINGERS, F.Cu at (-39.7, 36.4)
- added FID1: Fiducial, Fiducial:Fiducial_0.5mm_Mask1.5mm, F.Cu at (-51.9, 76.2)
- added FID2: Fiducial, Fiducial:Fiducial_0.5mm_Mask1.5mm, F.Cu at (-51.9, 79.3)
- added FID3: Fiducial, Fiducial:Fiducial_0.5mm_Mask1.5mm, F.Cu at (-48.8, 76.2)
- added FID4: Fiducial, Fiducial:Fiducial_0.5mm_Mask1.5mm, F.Cu at (-48.8, 79.3)
- added FID5: Fiducial, Fiducial:Fiducial_0.5mm_Mask1.5mm, F.Cu at (-45.8, 76.2)
- added FID6: Fiducial, Fiducial:Fiducial_0.5mm_Mask1.5mm, F.Cu at (-45.8, 79.3)
- added GNDTP1: TP, TestPoint:TestPoint_Pad_D1.5mm, F.Cu at (-55.2, 80.0)
- added J5: 12402012E212A, Library:AMPHENOL_12402012E212A, F.Cu at (168.3, 71.2)
- added L1: 4.7uH, LED_SMD:LED_0805_2012Metric, F.Cu at (-42.0, 53.1)
- added R1: 10k, Resistor_SMD:R_0603_1608Metric, F.Cu at (-54.9, 71.4)
- added R10: 100k, Resistor_SMD:R_0603_1608Metric, F.Cu at (-54.9, 49.3)
- added R11: 5k1, Resistor_SMD:R_0603_1608Metric, F.Cu at (-54.9, 51.9)
- added R12: 5k1, Resistor_SMD:R_0603_1608Metric, F.Cu at (-54.9, 54.4)
- added R13: 0R, Resistor_SMD:R_0603_1608Metric, F.Cu at (-50.9, 61.4)
- added R14: 0R, Resistor_SMD:R_0603_1608Metric, F.Cu at (-50.9, 63.9)
- added R17: 0R, Resistor_SMD:R_0603_1608Metric, F.Cu at (-50.9, 66.4)
- added R2: 10k, Resistor_SMD:R_0603_1608Metric, F.Cu at (-50.9, 58.9)
- added R20: 0R, Resistor_SMD:R_0603_1608Metric, F.Cu at (-50.9, 68.9)
- added R23: 0R, Resistor_SMD:R_0402_1005Metric, F.Cu at (-48.6, 43.5)
- added R25: 0R, Resistor_SMD:R_0402_1005Metric, F.Cu at (-48.6, 45.5)
- added R26: 0R, Resistor_SMD:R_0402_1005Metric, F.Cu at (-48.6, 47.5)
- added R27: 0R, Resistor_SMD:R_0402_1005Metric, F.Cu at (-48.6, 49.5)
- added R28: 0R, Resistor_SMD:R_0402_1005Metric, F.Cu at (-45.7, 43.5)
- added R29: 0R, Resistor_SMD:R_0402_1005Metric, F.Cu at (-45.7, 45.5)
- added R3: 1k, Resistor_SMD:R_0603_1608Metric, F.Cu at (-54.9, 41.8)
- added R30: 0R, Resistor_SMD:R_0402_1005Metric, F.Cu at (-45.7, 47.5)
- added R31: 0R, Resistor_SMD:R_0402_1005Metric, F.Cu at (-45.7, 49.5)
- added R4: 1k, Resistor_SMD:R_0603_1608Metric, F.Cu at (-54.9, 44.3)
- added R5: 1k, Resistor_SMD:R_0603_1608Metric, F.Cu at (-54.9, 46.8)
- added R6: 0R, Resistor_SMD:R_0402_1005Metric, F.Cu at (-51.5, 43.5)
- added R7: 4.35k, Resistor_SMD:R_0402_1005Metric, F.Cu at (-51.5, 45.5)
- added R8: 10k, Resistor_SMD:R_0402_1005Metric, F.Cu at (-51.5, 47.5)
- added R9: 0R, Resistor_SMD:R_0402_1005Metric, F.Cu at (-51.5, 49.5)
- added SW1: 2425754-1, Library:2425754-1_TEC, F.Cu at (88.8, 57.3)
- added SW2: 2425754-1, Library:2425754-1_TEC, F.Cu at (88.8, 70.9)
- added SW3: 2425754-1, Library:2425754-1_TEC, F.Cu at (88.8, 84.6)
- added TP1: TestPoint, TestPoint:TestPoint_Pad_D1.5mm, F.Cu at (-55.2, 83.6)
- added U3: PTS645SK43SMTR92LFS, Library:SWITCH_45SK43SMTR92LFS, B.Cu at (140.8, 90.2)
- added U4: PTS645SK43SMTR92LFS, Library:SWITCH_45SK43SMTR92LFS, B.Cu at (133.1, 90.2)
- added U5: PTS645SK43SMTR92LFS, Library:SWITCH_45SK43SMTR92LFS, B.Cu at (122.8, 55.7)
- added U6: PTS645SK43SMTR92LFS, Library:SWITCH_45SK43SMTR92LFS, B.Cu at (130.5, 55.7)
- added U7: PTS645SK43SMTR92LFS, Library:SWITCH_45SK43SMTR92LFS, B.Cu at (138.1, 55.7)

Commit message: Premier changement
Alice
Parts:
- moved J5 3.91 mm to (164.4, 71.5)
Changed lines of the file:
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@@
 	(footprint "Library:AMPHENOL_12402012E212A"
 		(layer "F.Cu")
-		(at 168.26 71.2 90)
+		(at 164.36 71.5 90)
 		(tags "usb")
 		(property "Reference" "J5"
@@
 			(keep_text_aligned yes)
 		)
-		(gr_text "85.0000 mm"
+		(gr_text "85,0000 mm"
 			(locked yes)
 			(at 129 32.35 0)
@@
 			(keep_text_aligned yes)
 		)
-		(gr_text "50.0000 mm"
+		(gr_text "50,0000 mm"
 			(locked yes)
 			(at 63.35 73.3 90)
