File: CreditCard/CreditCard.kicad_pcb (KiCad board)
At the start: 2 copper layers, 85 x 50 mm, 82 parts, among them J1 2060-1452/998-404, J2 MEM2052-00-195-00-A_REVA, J5 12402012E212A, SW1 2425754-1, SW2 2425754-1, SW3 2425754-1, U1 BQ24230RGTR, U10 PAM8403DR, U2 MCP1603T-330I/OS, U3 PTS645SK43SMTR92LFS, U4 PTS645SK43SMTR92LFS, U5 PTS645SK43SMTR92LFS, U6 PTS645SK43SMTR92LFS, U7 PTS645SK43SMTR92LFS, U8 ESP32-C6-WROOM-1U-N4, U9 SPKM.36.8.B, Y1 MS1V-T1K-32.768KHZ-12.5PF-20P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

Commit message: a toi de jouer
Manque:
schema pour l'ampli et speaker
rooting :)
Parts:
- removed 3VTP1, GNDTP1: TP, TestPoint:TestPoint_Pad_D1.5mm
- removed C1, C10, C11, C18, C19, C20, C21, C8, C9: 0.1uF, Capacitor_SMD:C_0603_1608Metric
- removed C12, C17: 12pF, Capacitor_SMD:C_0603_1608Metric
- removed C13, C15, C3, C4: 4.7uF, Capacitor_SMD:C_0805_2012Metric
- removed C14, C2: 1uF, Capacitor_SMD:C_0603_1608Metric
- removed C16: 100n, Capacitor_SMD:C_0603_1608Metric
- removed C7: 22uF, Capacitor_SMD:C_1206_3216Metric
- removed D1, D2, D3: LED, LED_SMD:LED_0805_2012Metric
- removed D5: D_TVS, Diode_SMD:D_SOD-323_HandSoldering
- removed F1, F2, F4, F5, F6, F7, F8: ~, CommonLib_HORUS:GOLD_FINGERS
- removed FID1, FID2, FID3, FID4, FID5, FID6: Fiducial, Fiducial:Fiducial_0.5mm_Mask1.5mm
- removed J1: 2060-1452/998-404, Library:CONN2_2059-302&slash_998-403_WAG
- removed J2: MEM2052-00-195-00-A_REVA, Library:GCT_MEM2052-00-195-00-A_REVA
- removed J5: 12402012E212A, Library:AMPHENOL_12402012E212A
- removed L1: 4.7uH, LED_SMD:LED_0805_2012Metric
- removed R1, R2: 10k, Resistor_SMD:R_0603_1608Metric
- removed R10: 100k, Resistor_SMD:R_0603_1608Metric
- removed R11, R12: 5k1, Resistor_SMD:R_0603_1608Metric
- removed R13, R14, R17, R20: 0R, Resistor_SMD:R_0603_1608Metric
- removed R23, R25, R26, R27, R28, R29, R30, R31, R6, R9: 0R, Resistor_SMD:R_0402_1005Metric
- removed R3, R4, R5: 1k, Resistor_SMD:R_0603_1608Metric
- removed R7: 4.35k, Resistor_SMD:R_0402_1005Metric
- removed R8: 10k, Resistor_SMD:R_0402_1005Metric
- removed S1: EG1271A, Library:SW_EG1271A
- removed SW1, SW2, SW3: 2425754-1, Library:2425754-1_TEC
- removed TP1: TestPoint, TestPoint:TestPoint_Pad_D1.5mm
- removed U1: BQ24230RGTR, Library:RGT16_1P7X1P7
- removed U10: PAM8403DR, Library:SOIC_8403DR_DIO
- removed U2: MCP1603T-330I/OS, Library:TSOT5_MC_MCH
- removed U3, U4, U5, U6, U7: PTS645SK43SMTR92LFS, Library:SWITCH_45SK43SMTR92LFS
- removed U8: ESP32-C6-WROOM-1U-N4, Library:XCVR_ESP32-C6-WROOM-1U-N4
- removed U9: SPKM.36.8.B, Library:SPEAKER
- removed Y1: MS1V-T1K-32.768KHZ-12.5PF-20PPM-TA-QC, Library:XTAL_MS1V-T1K-32.768KHZ-12.5PF-20PPM-TA-QC
Other:
- board size 85 x 50 mm -> 50.8 x 88.9 mm

Commit message: Goldfinger
Alice la queen
Parts:
- added 3VTP1: TP, TestPoint:TestPoint_Pad_D1.5mm, F.Cu at (-80.8, 48.1)
- added C1: 0.1uF, Capacitor_SMD:C_0603_1608Metric, F.Cu at (-21.8, 25.4)
- added C10: 0.1uF, Capacitor_SMD:C_0603_1608Metric, F.Cu at (-63.9, 27.6)
- added C11: 0.1uF, Capacitor_SMD:C_0603_1608Metric, F.Cu at (-63.9, 30.1)
- added C12: 12pF, Capacitor_SMD:C_0603_1608Metric, F.Cu at (-21.8, 32.9)
- added C13: 4.7uF, Capacitor_SMD:C_0805_2012Metric, F.Cu at (-44.8, 61.1)
- added C14: 1uF, Capacitor_SMD:C_0603_1608Metric, F.Cu at (-49.1, 45.2)
- added C15: 4.7uF, Capacitor_SMD:C_0805_2012Metric, F.Cu at (-44.8, 64.1)
- added C16: 100n, Capacitor_SMD:C_0603_1608Metric, F.Cu at (-49.1, 47.7)
- added C17: 12pF, Capacitor_SMD:C_0603_1608Metric, F.Cu at (-21.8, 35.4)
- added C18: 0.1uF, Capacitor_SMD:C_0603_1608Metric, F.Cu at (-63.9, 32.6)
- added C19: 0.1uF, Capacitor_SMD:C_0603_1608Metric, F.Cu at (-63.9, 35.1)
- added C2: 1uF, Capacitor_SMD:C_0603_1608Metric, F.Cu at (-21.8, 27.9)
- added C20: 0.1uF, Capacitor_SMD:C_0603_1608Metric, F.Cu at (-63.9, 37.6)
- added C21: 0.1uF, Capacitor_SMD:C_0603_1608Metric, F.Cu at (-63.9, 40.1)
- added C3: 4.7uF, Capacitor_SMD:C_0805_2012Metric, F.Cu at (-44.8, 55.1)
- added C4: 4.7uF, Capacitor_SMD:C_0805_2012Metric, F.Cu at (-44.8, 58.1)
- added C7: 22uF, Capacitor_SMD:C_1206_3216Metric, F.Cu at (-28.5, 60.6)
- added C8: 0.1uF, Capacitor_SMD:C_0603_1608Metric, F.Cu at (-49.1, 42.7)
- added C9: 0.1uF, Capacitor_SMD:C_0603_1608Metric, F.Cu at (-21.8, 30.4)
- added D1: LED, LED_SMD:LED_0805_2012Metric, F.Cu at (-44.8, 42.9)
- added D2: LED, LED_SMD:LED_0805_2012Metric, F.Cu at (-44.8, 46.0)
- added D3: LED, LED_SMD:LED_0805_2012Metric, F.Cu at (-44.8, 49.0)
- added D5: D_TVS, Diode_SMD:D_SOD-323_HandSoldering, F.Cu at (-30.3, 50.8)
- added F1: ~, Library:GOLD_FINGERS, F.Cu at (-43.9, 27.3)
- added F2: ~, Library:GOLD_FINGERS, F.Cu at (-43.9, 29.6)
- added F3: ~, Library:GOLD_FINGERS, F.Cu at (-43.9, 31.8)
- added F4: ~, Library:GOLD_FINGERS, F.Cu at (-43.9, 34.1)
- added F5: ~, Library:GOLD_FINGERS, F.Cu at (-67.0, 71.2)
- added F6: ~, Library:GOLD_FINGERS, F.Cu at (-67.0, 73.5)
- added FID1: Fiducial, Fiducial:Fiducial_0.5mm_Mask1.5mm, F.Cu at (-77.5, 47.8)
- added FID2: Fiducial, Fiducial:Fiducial_0.5mm_Mask1.5mm, F.Cu at (-77.5, 50.9)
- added FID3: Fiducial, Fiducial:Fiducial_0.5mm_Mask1.5mm, F.Cu at (-74.5, 47.8)
- added FID4: Fiducial, Fiducial:Fiducial_0.5mm_Mask1.5mm, F.Cu at (-74.5, 50.9)
- added FID5: Fiducial, Fiducial:Fiducial_0.5mm_Mask1.5mm, F.Cu at (-71.4, 47.8)
- added FID6: Fiducial, Fiducial:Fiducial_0.5mm_Mask1.5mm, F.Cu at (-71.4, 50.9)
- added GNDTP1: TP, TestPoint:TestPoint_Pad_D1.5mm, F.Cu at (-80.8, 51.6)
- added J1: 2060-1452/998-404, Library:CONN2_2059-302&slash_998-403_WAG, F.Cu at (-36.6, 46.8)
- added J2: MEM2052-00-195-00-A_REVA, Library:GCT_MEM2052-00-195-00-A_REVA, F.Cu at (-43.0, 12.2)
- added J5: 12402012E212A, Library:AMPHENOL_12402012E212A, F.Cu at (-37.0, 58.8)
- added L1: 4.7uH, LED_SMD:LED_0805_2012Metric, F.Cu at (-44.8, 52.0)
- added R1: 10k, Resistor_SMD:R_0603_1608Metric, F.Cu at (-21.8, 37.9)
- added R10: 100k, Resistor_SMD:R_0603_1608Metric, F.Cu at (-49.1, 57.7)
- added R11: 5k1, Resistor_SMD:R_0603_1608Metric, F.Cu at (-49.1, 60.2)
- added R12: 5k1, Resistor_SMD:R_0603_1608Metric, F.Cu at (-49.1, 62.7)
- added R13: 0R, Resistor_SMD:R_0603_1608Metric, F.Cu at (-17.8, 27.9)
- added R14: 0R, Resistor_SMD:R_0603_1608Metric, F.Cu at (-17.8, 30.4)
- added R17: 0R, Resistor_SMD:R_0603_1608Metric, F.Cu at (-17.8, 32.9)
- added R2: 10k, Resistor_SMD:R_0603_1608Metric, F.Cu at (-17.8, 25.4)
- added R20: 0R, Resistor_SMD:R_0603_1608Metric, F.Cu at (-17.8, 35.4)
- added R23: 0R, Resistor_SMD:R_0402_1005Metric, F.Cu at (-28.5, 42.4)
- added R25: 0R, Resistor_SMD:R_0402_1005Metric, F.Cu at (-28.5, 44.4)
- added R26: 0R, Resistor_SMD:R_0402_1005Metric, F.Cu at (-28.5, 46.4)
- added R27: 0R, Resistor_SMD:R_0402_1005Metric, F.Cu at (-28.5, 48.4)
- added R28: 0R, Resistor_SMD:R_0402_1005Metric, F.Cu at (-25.6, 42.4)
- added R29: 0R, Resistor_SMD:R_0402_1005Metric, F.Cu at (-25.6, 44.4)
- added R3: 1k, Resistor_SMD:R_0603_1608Metric, F.Cu at (-49.1, 50.2)
- added R30: 0R, Resistor_SMD:R_0402_1005Metric, F.Cu at (-25.6, 46.4)
- added R31: 0R, Resistor_SMD:R_0402_1005Metric, F.Cu at (-25.6, 48.4)
- added R4: 1k, Resistor_SMD:R_0603_1608Metric, F.Cu at (-49.1, 52.7)
- added R5: 1k, Resistor_SMD:R_0603_1608Metric, F.Cu at (-49.1, 55.2)
- added R6: 0R, Resistor_SMD:R_0402_1005Metric, F.Cu at (-31.4, 42.4)
- added R7: 4.35k, Resistor_SMD:R_0402_1005Metric, F.Cu at (-31.4, 44.4)
- added R8: 10k, Resistor_SMD:R_0402_1005Metric, F.Cu at (-31.4, 46.4)
- added R9: 0R, Resistor_SMD:R_0402_1005Metric, F.Cu at (-31.4, 48.4)
- added S1: EG1271A, Library:SW_EG1271A, F.Cu at (-37.6, 65.7)
- added SW1: 2425754-1, Library:2425754-1_TEC, F.Cu at (-80.2, 7.67)
- added SW2: 2425754-1, Library:2425754-1_TEC, F.Cu at (-80.2, 21.3)
- added SW3: 2425754-1, Library:2425754-1_TEC, F.Cu at (-80.2, 35.0)
- added TP1: TestPoint, TestPoint:TestPoint_Pad_D1.5mm, F.Cu at (-80.8, 55.2)
- added U1: BQ24230RGTR, Library:RGT16_1P7X1P7, F.Cu at (-28.3, 55.8)
- added U10: PAM8403DR, Library:SOIC_8403DR_DIO, F.Cu at (-57.6, 32.1)
- added U2: MCP1603T-330I/OS, Library:TSOT5_MC_MCH, F.Cu at (-28.8, 64.5)
- added U3: PTS645SK43SMTR92LFS, Library:SWITCH_45SK43SMTR92LFS, F.Cu at (-29.4, 27.9)
- added U4: PTS645SK43SMTR92LFS, Library:SWITCH_45SK43SMTR92LFS, F.Cu at (-29.4, 35.6)
- added U5: PTS645SK43SMTR92LFS, Library:SWITCH_45SK43SMTR92LFS, F.Cu at (-60.3, 7.18)
- added U6: PTS645SK43SMTR92LFS, Library:SWITCH_45SK43SMTR92LFS, F.Cu at (-60.3, 14.8)
- added U7: PTS645SK43SMTR92LFS, Library:SWITCH_45SK43SMTR92LFS, F.Cu at (-60.3, 22.5)
- added U8: ESP32-C6-WROOM-1U-N4, Library:XCVR_ESP32-C6-WROOM-1U-N4, F.Cu at (-23.5, 13.7)
- added U9: SPKM.36.8.B, Library:SPEAKER, F.Cu at (-59.3, 38.7)
- added Y1: MS1V-T1K-32.768KHZ-12.5PF-20PPM-TA-QC, Library:XTAL_MS1V-T1K-32.768KHZ-12.5PF-20PPM-TA-QC, F.Cu at (-48.5, 31.0)

Commit message: connection du audio amp
Parts:
- added C22: 4.7uF, Capacitor_SMD:C_0603_1608Metric, F.Cu at (-5.72, 10.9)
- added C23: 0.1uF, Capacitor_SMD:C_0603_1608Metric, F.Cu at (-5.72, 13.4)
- added C24: 470uf, Capacitor_SMD:C_0603_1608Metric, F.Cu at (-5.72, 15.9)
- added C25: 1uf, Capacitor_SMD:C_0603_1608Metric, F.Cu at (-1.72, 5.86)
- added C26: 0.1uF, Capacitor_SMD:C_0603_1608Metric, F.Cu at (-1.72, 8.37)
- added C5: 0.1uF, Capacitor_SMD:C_0603_1608Metric, F.Cu at (-5.72, 5.86)
- added C6: 4.7uF, Capacitor_SMD:C_0603_1608Metric, F.Cu at (-5.72, 8.37)
- added R15: 18k, Resistor_SMD:R_0603_1608Metric, F.Cu at (-1.72, 10.9)
- added R16: 18k, Resistor_SMD:R_0603_1608Metric, F.Cu at (-1.72, 13.4)
- added R18: 0, Resistor_SMD:R_0603_1608Metric, F.Cu at (-1.72, 15.9)
- added U11: SPKM.36.8.B, Library:SPEAKER, F.Cu at (2.92, 5.36)
Connections:
- U10 pad 1: unconnected-(U10-+OUT_L-Pad1) -> Net-(U10-+OUT_L)
- U10 pad 10: unconnected-(U10-INR-Pad10) -> Net-(U10-INR)
- U10 pad 11: unconnected-(U10-GND-Pad11) -> GND
- U10 pad 12: unconnected-(U10-SHND-Pad12) -> AudioCS
- U10 pad 13: unconnected-(U10-PVDD-Pad13) -> 3V3
- U10 pad 14: unconnected-(U10--OUT_R-Pad14) -> Net-(U10--OUT_R)
- U10 pad 15: unconnected-(U10-PGND-Pad15) -> GND
- U10 pad 16: unconnected-(U10-+OUT_R-Pad16) -> Net-(U10-+OUT_R)
- U10 pad 2: unconnected-(U10-PGND-Pad2) -> GND
- U10 pad 3: unconnected-(U10--OUT_L-Pad3) -> Net-(U10--OUT_L)
- U10 pad 4: unconnected-(U10-PVDD-Pad4) -> 3V3
- U10 pad 5: unconnected-(U10-MUTE-Pad5) -> Net-(U10-MUTE)
- U10 pad 6: unconnected-(U10-VDD-Pad6) -> 3V3
- U10 pad 7: unconnected-(U10-INL-Pad7) -> Net-(U10-INL)
- U10 pad 8: unconnected-(U10-VREF-Pad8) -> Net-(U10-VREF)
- U8 pad 11: SCK -> AudioL
- U8 pad 12: unconnected-(U8-IO11-Pad12) -> AudioR
- U8 pad 18: unconnected-(U8-IO20-Pad18) -> AudioCS
- U8 pad 23: unconnected-(U8-IO15-Pad23) -> SCK
- U9 pad 1: unconnected-(U9-VDD-Pad1) -> Net-(U10-+OUT_R)
- U9 pad 2: unconnected-(U9-GND-Pad2) -> Net-(U10--OUT_R)

Commit message: aliiice
Parts:
- removed F1, F2: ~, Library:GOLD_FINGERS
- added R19: 0, Resistor_SMD:R_0603_1608Metric, F.Cu at (145.6, 49.8)
- added R21: 0, Resistor_SMD:R_0603_1608Metric, F.Cu at (145.6, 52.3)
- C1, C16, C9, D5, F3, F4, J5, R10, R13, U3, U4, U8: moved to B.Cu
- J2: value MEM2052-00-195-00-A_REVA -> LCD; footprint Library:GCT_MEM2052-00-195-00-A_REVA -> Library:LCD
- moved SW3 233.6 mm to (136.3, 122.9), turned to 90 degrees
- moved SW2 226.8 mm to (122.6, 122.9), turned to 90 degrees
- moved SW1 221.5 mm to (109.0, 122.9), turned to 90 degrees
- moved C16 199.6 mm to (148.5, 76.0), turned to 180 degrees
- moved R10 198.6 mm to (148.5, 78.0), turned to 180 degrees
- moved U7 197.8 mm to (136.5, 42.0)
- moved U6 187.8 mm to (125.5, 42.0)
- moved J5 185.2 mm to (147.5, 42.0), turned to -90 degrees
- moved S1 184.6 mm to (147.0, 67.0), turned to 90 degrees
- moved D5 179.7 mm to (148.0, 73.5), turned to 180 degrees
- moved U5 178.3 mm to (114.5, 42.0)
- moved J2 178.1 mm to (113.6, 97.0)
- moved F3 162.7 mm to (113.5, 73.0), turned to 180 degrees
- moved U8 158.9 mm to (119.0, 84.0), turned to 180 degrees
- moved F4 158.8 mm to (110.0, 73.0), turned to 180 degrees
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Connections:
- U8 pad 19: CardDetect_SD -> LCD_CS
- U8 pad 24: SDA -> LCD_D/C
- U8 pad 25: SCL -> LCD_RESET

Commit message: aliiice fin de journée
Parts:
- removed J5: 12402012E212A, Library:AMPHENOL_12402012E212A
- added J3: 12402012E212A, Library:AMPHENOL_12402012E212A, B.Cu at (147.0, 85.2)
- added MEC1: ~, Library:Mounting_3mm, F.Cu at (173.5, 42.0)
- added MEC2: ~, Library:Mounting_3mm, F.Cu at (173.5, 45.6)
- added MEC3: ~, Library:Mounting_3mm, F.Cu at (173.5, 48.8)
- added MEC4: ~, Library:Mounting_3mm, F.Cu at (173.5, 52.0)
- C12, C17, C2, C22, C23, C24, C25, C26, C5, C6, R1, R14, R15, R16, R17, R18, R2, R20, U10, U11, U9, Y1: moved to B.Cu
- moved U9 170.6 mm to (103.0, 91.4), turned to 180 degrees
- moved U10 170.3 mm to (104.2, 85.4), turned to 180 degrees
- moved Y1 152.3 mm to (102.5, 51.0), turned to 180 degrees
- moved C22 144.9 mm to (106.2, 103.0), turned to 180 degrees
- moved C23 144.9 mm to (106.2, 105.5), turned to 180 degrees
- moved C5 144.9 mm to (106.2, 98.0), turned to 180 degrees
- moved C24 144.9 mm to (106.2, 108.0), turned to 180 degrees
- moved C6 144.9 mm to (106.2, 100.5), turned to 180 degrees
- moved C25 138.8 mm to (102.2, 98.0), turned to 180 degrees
- moved C26 138.8 mm to (102.2, 100.5), turned to 180 degrees
- moved R15 138.8 mm to (102.2, 103.0), turned to 180 degrees
- moved R16 138.8 mm to (102.2, 105.5), turned to 180 degrees
- moved R18 138.8 mm to (102.2, 108.0), turned to 180 degrees
- moved U11 133.7 mm to (103.0, 94.0), turned to 180 degrees
- moved C17 128.9 mm to (105.7, 54.0), turned to -90 degrees
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
Commit message: rooting presque fini
Parts:
- removed R13, R14, R17, R20: 0R, Resistor_SMD:R_0603_1608Metric
- removed R25, R27, R28, R30, R6, R9: 0R, Resistor_SMD:R_0402_1005Metric
- C10, C11, C13, C14, C15, C18, C3, C4, C7, C8, D2, D3, J1, L1, R11, R12, R23, R26, R29, R31, R4, R5, R7, R8, U1, U2: moved to B.Cu
- C2, C22, C23, C24, C25, C26, C5, C6, R1, R15, R16, R18, R2, U10, U11, U9: moved to F.Cu
- moved C18 220.8 mm to (138.8, 120.2)
- moved C11 209.5 mm to (125.2, 120.2)
- moved C21 203.9 mm to (140.0, 37.6)
- moved C10 198.5 mm to (111.6, 120.2)
- moved R3 197.9 mm to (148.6, 59.6), turned to 90 degrees
- moved D1 193.8 mm to (148.6, 55.8), turned to -90 degrees
- moved C8 193.7 mm to (142.8, 69.0)
- moved C20 192.9 mm to (129.0, 37.6)
- moved C4 187.8 mm to (142.8, 66.8)
- moved L1 183.8 mm to (138.4, 66.8)
- moved C19 181.9 mm to (118.0, 37.6)
- moved C3 180.9 mm to (136.0, 58.8), turned to 180 degrees
- moved R5 179.7 mm to (130.6, 60.7), turned to 90 degrees
- moved R4 177.1 mm to (127.8, 62.9)
- moved D3 174.2 mm to (129.2, 57.9)
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Connections:
- C12 pad 1: Net-(C12-Pad1) -> XTAL_P
- C17 pad 1: Net-(C17-Pad1) -> XTAL_N
- Y1 pad 1: Net-(C12-Pad1) -> XTAL_P
- Y1 pad 2: Net-(C17-Pad1) -> XTAL_N
Routing:
- net 3V3: track 0.00 -> 66.1 mm, vias 0 -> 2
- net Vsys: track 0.00 -> 37.0 mm
- net GND: track 0.00 -> 36.6 mm, vias 0 -> 1
- net MCU_EN: track 0.00 -> 24.6 mm, vias 0 -> 1
- net Vbus: track 0.00 -> 17.5 mm, vias 0 -> 2
- net Vbat: track 0.00 -> 15.8 mm
- net IO9: track 0.00 -> 13.9 mm
- net GPIO7: track 0.00 -> 10.1 mm
- net GPIO6: track 0.00 -> 10.1 mm
- net GPIO5: track 0.00 -> 10.1 mm
- net /PWR/TD_CHR: track 0.00 -> 8.15 mm
- net XTAL_N: track 0.00 -> 7.72 mm
- net XTAL_P: track 0.00 -> 7.72 mm
- net Net-(U8-IO8): track 0.00 -> 7.27 mm, vias 0 -> 1
- net Net-(U10-+OUT_R): track 0.00 -> 6.38 mm
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Other:
- board text added: "LED-3V3"

Commit message: Alice hihi
Parts:
- C22, C23, C24, C25, C26, C5, C6, R15, R16, R18, U10, U11, U9: moved to B.Cu
- moved C25 68.2 mm to (117.0, 67.0), turned to 0 degrees
- moved C6 67.2 mm to (118.0, 72.5), turned to 0 degrees
- moved C26 66.1 mm to (116.2, 70.5), turned to 180 degrees
- moved R18 64.4 mm to (117.0, 68.8), turned to 180 degrees
- moved R15 62.3 mm to (114.5, 72.2), turned to 0 degrees
- moved U11 59.8 mm to (112.5, 65.0)
- moved C5 52.6 mm to (110.9, 75.5), turned to 180 degrees
- moved U10 48.6 mm to (108.8, 69.1), turned to 180 degrees
- moved C23 35.2 mm to (102.5, 69.0), turned to 180 degrees
- moved C24 35.2 mm to (102.5, 70.8), turned to 180 degrees
- moved R16 35.2 mm to (102.5, 72.5), turned to 0 degrees
- moved C22 34.7 mm to (102.7, 75.1)
- moved U9 34.1 mm to (102.5, 66.0)
- moved J2 9.73 mm to (110.3, 87.8)
Routing:
- net Net-(U10--OUT_L): track 6.12 -> 2.29 mm
- net Net-(U10-+OUT_L): track 6.30 -> 2.48 mm
- net Net-(U10-+OUT_R): track 6.38 -> 2.56 mm
- net Net-(U10--OUT_R): track 6.19 -> 2.63 mm
- net 3V3: track 66.1 -> 63.0 mm
- net Net-(C6-Pad1): track 0.00 -> 2.35 mm
- net Net-(U10-INL): track 0.00 -> 2.19 mm
- net Net-(U10-VREF): track 0.00 -> 2.08 mm
- net Net-(C22-Pad1): track 0.00 -> 1.90 mm
- net Net-(U10-INR): track 0.00 -> 1.78 mm
- net Net-(U10-MUTE): track 5.62 -> 5.06 mm

Commit message: continuité rooting
add diff pair dn-dp
add sw on-off on pcb
Parts:
- moved C16 70.0 mm to (143.5, 45.4)
- moved D5 70.0 mm to (139.7, 46.0)
- moved R10 70.0 mm to (141.7, 45.4)
- moved S1 70.0 mm to (147.1, 46.2)
- moved J2 9.63 mm to (113.6, 96.9)
Routing:
- net D_N: track 0.00 -> 55.7 mm
- net D_P: track 0.00 -> 55.4 mm, vias 0 -> 2
- net Net-(F6-GOLDFINGER): track 4.41 -> 5.03 mm
