File: CreditCard/_autosave-CreditCard.kicad_pcb (KiCad board)
At the start: 2 copper layers, 85 x 50 mm, 82 parts, among them J1 2060-1452/998-404, J2 MEM2052-00-195-00-A_REVA, J5 12402012E212A, SW1 2425754-1, SW2 2425754-1, SW3 2425754-1, U1 BQ24230RGTR, U10 PAM8403DR, U2 MCP1603T-330I/OS, U3 PTS645SK43SMTR92LFS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

Commit message: manque écran
manque seulement l'écran le reste est ajouter
Parts:
- moved TP1 107.0 mm to (-11.6, 35.4), turned to 180 degrees
- moved U1 104.1 mm to (-63.8, 27.2), turned to 180 degrees
- moved GNDTP1 101.7 mm to (-11.6, 39.0), turned to 180 degrees
- moved D5 101.3 mm to (-58.0, 26.9), turned to 180 degrees
- moved R31 100.8 mm to (-68.3, 30.9), turned to 180 degrees
- moved C7 99.8 mm to (-52.6, 26.7), turned to 180 degrees
- moved C15 99.4 mm to (-47.6, 26.5), turned to 180 degrees
- moved R27 98.4 mm to (-65.4, 30.9), turned to 180 degrees
- moved R30 97.2 mm to (-68.3, 32.9), turned to 180 degrees
- moved R12 96.8 mm to (-43.4, 27.8), turned to 180 degrees
- moved 3VTP1 96.6 mm to (-11.6, 42.5), turned to 180 degrees
- moved R9 96.2 mm to (-62.5, 30.9), turned to 180 degrees
- moved FID2 96.1 mm to (-14.9, 39.7), turned to 180 degrees
- moved R26 94.7 mm to (-65.4, 32.9), turned to 180 degrees
- moved R29 93.7 mm to (-68.3, 34.9), turned to 180 degrees
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