File: CreditCard/PWR.kicad_sch (KiCad schematic)
At the start: 38 parts, among them J1 2059-302/998-403, J5 12402012E212A, U1 BQ24230RGTR, U2 MCP1603T-330I/OS

Commit message: manque écran
manque seulement l'écran le reste est ajouter
Parts:
- removed J1: 2059-302/998-403, LIB:CONN2_2059-302&slash_998-403_WAG, symbol LIB:2059-302_998-403
- removed S2: EG1271A, LIB:SW_EG1271A, symbol LIB:EG1271A
- removed U1: BQ24230RGTR, LIB:RGT16_1P7X1P7, symbol 2024-07-09_01-17-53:BQ24230RGTR
- removed U2: MCP1603T-330I/OS, LIB:TSOT5_MC_MCH, symbol LIB:MCP1603T-330I_OS
- added J1: 2060-1452/998-404, Library:CONN2_2059-302&slash_998-403_WAG, symbol Library:2060-1452_998-404
- added S1: EG1271A, Library:SW_EG1271A, symbol Library:EG1271A
- added U1: BQ24230RGTR, Library:RGT16_1P7X1P7, symbol Library:BQ24230RGTR
- added U2: MCP1603T-330I/OS, Library:TSOT5_MC_MCH, symbol Library:MCP1603T-330I_OS
Connections:
- net 3V3: now also U2.4 (VFB/VOUT)
- net CE_CHR: now also U1.4 (*CE)
- net EN1_CHR: now also U1.6 (EN1)
- net EN2_CHR: now also U1.5 (EN2)
- net GND: now also J1.1 (1_1), J1.2 (1_2), S1.3, S1.6, U1.17 (EPAD), U1.8 (VSS), U2.2 (GND)
- net ILIM_CHR: now also U1.12 (ILIM)
- net IO_CHG: now also U1.9 (*CHG)
- net ISET_CHR: now also U1.16 (ISET)
- net POWER_EN: now also S1.2, S1.5, U2.3 (*SHDN)
- net TD_CHR: now also U1.15 (TD)
- net TMR_CHR: now also U1.14 (TMR)
- net TS_CHR: now also U1.1 (TS)
- net Vbat: now also J1.3 (2_1), J1.4 (2_2), U1.2 (BAT), U1.3 (BAT)
- net Vbus: now also U1.13 (IN)
- net Vsys: now also S1.1, S1.4, U1.10 (OUT), U1.11 (OUT), U2.1 (VIN)
- net at D3.1 (K): now also U1.7 (*PGOOD)
- net at L1.1: now also U2.5 (LX)
Other:
- moved on the sheet: L1

Commit message: Goldfinger
Alice la queen
Parts:
- removed F7, F8: ~, CommonLib_HORUS:GOLD_FINGERS, symbol LIB:GoldFingers
- added F5, F6: ~, Library:GOLD_FINGERS, symbol Library:GoldFingers
Connections:
- net at J5.A8 (SBU1): now also F6.1 (GOLDFINGER)
- net at J5.B8 (SBU2): now also F5.1 (GOLDFINGER)

Commit message: ajout .step usbc
Parts:
- removed J5: 12402012E212A, Library:AMPHENOL_12402012E212A, symbol Library:12402012E212A
- added J3: 12402012E212A, Library:AMPHENOL_12402012E212A, symbol Library:12402012E212A
Connections:
- net D_N: now also J3.A7 (D-_A), J3.B7 (D-_B)
- net D_P: now also J3.A6 (D+_A), J3.B6 (D+_B)
- net GND: now also J3.A1_B12 (GND), J3.B1_A12 (GND__1), J3.SH1 (SHIELD), J3.SH2 (SHIELD__1), J3.SH3 (SHIELD__2), J3.SH4 (SHIELD__3)
- net Vbus: now also J3.A4_B9 (VBUS)
- net at F6.1 (GOLDFINGER): now also J3.A8 (SBU1)
- net at R12.2: now also J3.A5 (CC1_A)
- net at R11.1: now also J3.B5 (CC1_B)
- net at F5.1 (GOLDFINGER): now also J3.B8 (SBU2)
